Commit message: Rotation of model robot

File: urdf/heron_urdf.urdf (robot description, URDF)
Before this commit: robot heron_urdf, 5 links, 4 joints
Joints:
- joint wheel_BL: origin xyz=0.154955093786635 0.05 -0.0610768464243845 rpy=1.5707963267949 1.5707963267949 0 -> xyz=-0.050044906213365 0.161235 0.0389231535756156 rpy=1.5707963267949 1.5707963267949 -1.5707963267949
- joint wheel_BR: origin xyz=-0.205044906213365 0.05 -0.0610768464243845 rpy=1.5707963267949 1.5707963267949 0 -> xyz=-0.050044906213365 -0.211235 0.0389231535756156 rpy=1.5707963267949 1.5707963267949 1.5707963267949
- joint wheel_FL: origin xyz=0.154955093786635 -0.35 -0.0610768464243844 rpy=1.5707963267949 1.5707963267949 0 -> xyz=0.349955093786635 0.161235 0.0389231535756156 rpy=1.5707963267949 1.5707963267949 -1.5707963267949
- joint wheel_FR: origin xyz=-0.205044906213365 -0.35 -0.0610768464243845 rpy=1.5707963267949 1.5707963267949 0 -> xyz=0.349955094 -0.211235 0.0389231535756156 rpy=1.5707963267949 1.5707963267949 1.5707963267949

Commit message: Test urdf robot

File: urdf/heron_urdf.urdf (robot description, URDF)
Before this commit: robot heron_urdf, 5 links, 4 joints
Joints:
- joint wheel_BL: origin xyz=-0.050044906213365 0.161235 0.0389231535756156 rpy=1.5707963267949 1.5707963267949 -1.5707963267949 -> xyz=-0.550044906213365 0.161235 0.0389231535756156 rpy=1.5707963267949 1.5707963267949 -1.5707963267949
- joint wheel_BR: origin xyz=-0.050044906213365 -0.211235 0.0389231535756156 rpy=1.5707963267949 1.5707963267949 1.5707963267949 -> xyz=-0.550044906213365 -0.211235 0.0389231535756156 rpy=1.5707963267949 1.5707963267949 1.5707963267949
- joint wheel_FL: origin xyz=0.349955093786635 0.161235 0.0389231535756156 rpy=1.5707963267949 1.5707963267949 -1.5707963267949 -> xyz=-0.150044906213365 0.161235 0.0389231535756156 rpy=1.5707963267949 1.5707963267949 -1.5707963267949
- joint wheel_FR: origin xyz=0.349955094 -0.211235 0.0389231535756156 rpy=1.5707963267949 1.5707963267949 1.5707963267949 -> xyz=-0.150044906213365 -0.211235 0.0389231535756156 rpy=1.5707963267949 1.5707963267949 1.5707963267949

Commit message: Update urdf for tf base_link

File: urdf/heron_urdf.urdf (robot description, URDF)
Before this commit: robot heron_urdf, 5 links, 4 joints
Joints:
- joint wheel_BL: origin xyz=-0.550044906213365 0.161235 0.0389231535756156 rpy=1.5707963267949 1.5707963267949 -1.5707963267949 -> xyz=-0.200044906213365 0.186235 0.0389231535756156 rpy=1.5707963267949 1.5707963267949 -1.5707963267949
- joint wheel_BR: origin xyz=-0.550044906213365 -0.211235 0.0389231535756156 rpy=1.5707963267949 1.5707963267949 1.5707963267949 -> xyz=-0.200044906213365 -0.186235 0.0389231535756156 rpy=1.5707963267949 1.5707963267949 1.5707963267949
- joint wheel_FL: origin xyz=-0.150044906213365 0.161235 0.0389231535756156 rpy=1.5707963267949 1.5707963267949 -1.5707963267949 -> xyz=0.199955093786635 0.186235 0.0389231535756156 rpy=1.5707963267949 1.5707963267949 -1.5707963267949
- joint wheel_FR: origin xyz=-0.150044906213365 -0.211235 0.0389231535756156 rpy=1.5707963267949 1.5707963267949 1.5707963267949 -> xyz=0.199955093786635 -0.186235 0.0389231535756156 rpy=1.5707963267949 1.5707963267949 1.5707963267949

Commit message: Partie supérieure implémentée

File: urdf/heron_urdf.urdf (robot description, URDF)
Before this commit: robot heron_urdf, 5 links, 4 joints
Links:
- added link plate, mass 0.389968906998643; collision mesh filename=package://heron/meshes/plate.STL; visual mesh filename=package://heron/meshes/plate.STL
- added link support, mass 0.389968906998643; collision mesh filename=package://heron/meshes/support.STL; visual mesh filename=package://heron/meshes/support.STL
Joints:
- added joint plate: type prismatic, parent base_link, child plate, origin xyz=-0.6642 -0.26 0.135 rpy=1.5707963267949 0 1.5707963267949, axis 0 1 0, limit lower=0.0 upper=0.386 effort=147 velocity=0.039
- added joint support: type fixed, parent base_link, child support, origin xyz=-0.2969 0.186235 0.004 rpy=1.5707963267949 0 -1.5707963267949
- joint wheel_BL: limit lower=0.0 upper=0.0 effort=9.1201845 velocity=8.79645942 -> (none); type revolute -> continuous
- joint wheel_BR: limit lower=0.0 upper=0.0 effort=9.1201845 velocity=8.79645942 -> (none); type revolute -> continuous
- joint wheel_FL: limit lower=0.0 upper=0.0 effort=9.1201845 velocity=8.79645942 -> (none); type revolute -> continuous
- joint wheel_FR: limit lower=0.0 upper=0.0 effort=9.1201845 velocity=8.79645942 -> (none); type revolute -> continuous

Commit message: Put the limit effort on the wheels

File: urdf/heron_urdf.urdf (robot description, URDF)
Before this commit: robot heron_urdf, 7 links, 6 joints
Joints:
- joint wheel_BL: limit (none) -> effort=9.1201845 velocity=8.79645942
- joint wheel_BR: limit (none) -> effort=9.1201845 velocity=8.79645942
- joint wheel_FL: limit (none) -> effort=9.1201845 velocity=8.79645942
- joint wheel_FR: limit (none) -> effort=9.1201845 velocity=8.79645942

Commit message: TF

File: urdf/heron_urdf.urdf (robot description, URDF)
Before this commit: robot heron_urdf, 7 links, 6 joints
Joints:
- joint plate: origin xyz=-0.6642 -0.26 0.135 rpy=1.5707963267949 0 1.5707963267949 -> (none)

Commit message: TF robot pieces

File: urdf/heron_urdf.urdf (robot description, URDF)
Before this commit: robot heron_urdf, 7 links, 6 joints
Joints:
- joint plate: origin (none) -> xyz=-0.6642 -0.26 0.035 rpy=1.5707963267949 0 1.5707963267949
- joint support: origin xyz=-0.2969 0.186235 0.004 rpy=1.5707963267949 0 -1.5707963267949 -> xyz=-0.2969 0.186235 -0.096 rpy=1.5707963267949 0 -1.5707963267949
- joint wheel_BL: origin xyz=-0.200044906213365 0.186235 0.0389231535756156 rpy=1.5707963267949 1.5707963267949 -1.5707963267949 -> xyz=-0.200044906213365 0.186235 -0.0610768464243844 rpy=1.5707963267949 1.5707963267949 -1.5707963267949
- joint wheel_BR: origin xyz=-0.200044906213365 -0.186235 0.0389231535756156 rpy=1.5707963267949 1.5707963267949 1.5707963267949 -> xyz=-0.200044906213365 -0.186235 -0.0610768464243844 rpy=1.5707963267949 1.5707963267949 1.5707963267949
- joint wheel_FL: origin xyz=0.199955093786635 0.186235 0.0389231535756156 rpy=1.5707963267949 1.5707963267949 -1.5707963267949 -> xyz=0.199955093786635 0.186235 -0.0610768464243844 rpy=1.5707963267949 1.5707963267949 -1.5707963267949
- joint wheel_FR: origin xyz=0.199955093786635 -0.186235 0.0389231535756156 rpy=1.5707963267949 1.5707963267949 1.5707963267949 -> xyz=0.199955093786635 -0.186235 -0.0610768464243844 rpy=1.5707963267949 1.5707963267949 1.5707963267949

Commit message: Update urdf to apply a tf on them

File: urdf/heron_urdf.urdf (robot description, URDF)
Before this commit: robot heron_urdf, 7 links, 6 joints
Joints:
- joint plate: origin xyz=-0.6642 -0.26 0.035 rpy=1.5707963267949 0 1.5707963267949 -> xyz=0 0 0 rpy=0 0 0
- joint support: origin xyz=-0.2969 0.186235 -0.096 rpy=1.5707963267949 0 -1.5707963267949 -> xyz=0 0 0 rpy=0 0 0

Commit message: TF updated and URDF too

File: urdf/heron_urdf.urdf (robot description, URDF)
Before this commit: robot heron_urdf, 7 links, 6 joints
Links:
- link wheel_BL: geometry collision mesh filename=package://heron/meshes/wheel_BL.dae scale=0.393700787 0.5 0.393700787; visual mesh filename=package://heron/meshes/wheel_BL.dae scale=0.393700787 0.5 0.393700787
- link wheel_BR: geometry collision mesh filename=package://heron/meshes/wheel_BR.dae scale=0.393700787 0.5 0.393700787; visual mesh filename=package://heron/meshes/wheel_BR.dae scale=0.393700787 0.5 0.393700787
- link wheel_FL: geometry collision mesh filename=package://heron/meshes/wheel_FL.dae scale=0.393700787 0.5 0.393700787; visual mesh filename=package://heron/meshes/wheel_FL.dae scale=0.393700787 0.5 0.393700787
- link wheel_FR: geometry collision mesh filename=package://heron/meshes/wheel_FR.dae scale=0.393700787 0.5 0.393700787; visual mesh filename=package://heron/meshes/wheel_FR.dae scale=0.393700787 0.5 0.393700787

Commit message: Update urdf

File: urdf/heron_urdf.urdf (robot description, URDF)
Before this commit: robot heron_urdf, 7 links, 6 joints
Joints:
- joint plate: axis 0 1 0 -> 0 0 1; origin xyz=0 0 0 rpy=0 0 0 -> xyz=-0.32 0 0.13 rpy=0 0 0
- joint support: origin xyz=0 0 0 rpy=0 0 0 -> xyz=-0.3 0 0 rpy=0 0 0
- joint wheel_BL: origin xyz=-0.200044906213365 0.186235 -0.0610768464243844 rpy=1.5707963267949 1.5707963267949 -1.5707963267949 -> xyz=-0.2 0.216235 -0.06 rpy=0 0 0
- joint wheel_BR: origin xyz=-0.200044906213365 -0.186235 -0.0610768464243844 rpy=1.5707963267949 1.5707963267949 1.5707963267949 -> xyz=-0.2 -0.216235 -0.06 rpy=0 0 0
- joint wheel_FL: origin xyz=0.199955093786635 0.186235 -0.0610768464243844 rpy=1.5707963267949 1.5707963267949 -1.5707963267949 -> xyz=0.2 -0.216235 -0.06 rpy=0 0 0
- joint wheel_FR: origin xyz=0.199955093786635 -0.186235 -0.0610768464243844 rpy=1.5707963267949 1.5707963267949 1.5707963267949 -> xyz=0.2 -0.216235 -0.06 rpy=0 0 0

Commit message: Change tf_robot for using joint_state_publisher

File: urdf/heron_urdf.urdf (robot description, URDF)
Before this commit: robot heron_urdf, 7 links, 6 joints
Joints:
- joint wheel_FL: origin xyz=0.2 -0.216235 -0.06 rpy=0 0 0 -> xyz=0.2 0.216235 -0.06 rpy=0 0 0

Commit message: Resolve winch height in meters and add base footpritn

File: urdf/heron_urdf.urdf (robot description, URDF)
Before this commit: robot heron_urdf, 7 links, 6 joints
Links:
- added link base_footprint; visual box size=0.001 0.001 0.001
Joints:
- added joint base_footprint: type fixed, parent base_footprint, child base_link, origin xyz=0 0 0.10 rpy=0 0 0
